File: project_template/my_Kicad10_Template_Rev4/my_Kicad10_Template_Rev4.kicad_pcb (KiCad board)
At the start: 2 copper layers, 0 parts

Commit message: docs: update project template
define : assembly layer
Other:
- board text added: "Board Specifications"
- board text added: "Bottom Assembly (Scale 1:1)"
- board text added: "Bottom Dimension (Scale 1:1)"
- board text added: "Bottom Testpoint (Scale 1:1)"
- board text added: "Top Assembly (Scale 1:1)"
- board text added: "Top Dimension (Scale 1:1)"
- board text added: "Top Testpoint (Scale 1:1)"
